Commit message: Final Project

File: body.urdf (robot description, URDF)
Before this commit: robot robot, 9 links, 8 joints
Links:
- removed link BackLeg
- removed link BackLowerLeg
- removed link FrontLeg
- removed link FrontLowerLeg
- removed link LeftLeg
- removed link LeftLowerLeg
- removed link RightLeg
- removed link RightLowerLeg
- added link BL, mass 1; collision box size=0.2 0.2 1; visual box size=0.2 0.2 1
- added link BR, mass 1; collision box size=0.2 0.2 1; visual box size=0.2 0.2 1
- added link BW, mass 1; collision box size=0.1 1.3 0.1; visual box size=0.1 1.3 0.1
- added link FL, mass 1; collision box size=0.2 0.2 1; visual box size=0.2 0.2 1
- added link FR, mass 1; collision box size=0.2 0.2 1; visual box size=0.2 0.2 1
- link Torso: geometry collision box size=1 2 0.5; visual box size=1 2 0.5
Joints:
- removed joint BackLeg_BackLowerLeg
- removed joint FrontLeg_FrontLowerLeg
- removed joint LeftLeg_LeftLowerLeg
- removed joint RightLeg_RightLowerLeg
- removed joint Torso_BackLeg
- removed joint Torso_FrontLeg
- removed joint Torso_LeftLeg
- removed joint Torso_RightLeg
- added joint Torso_BL: type revolute, parent Torso, child BL, origin xyz=-0.5 -0.9 1 rpy=0 0 0, axis 1 0 0, limit lower=-3.14159 upper=3.14159 effort=0.0 velocity=0.0
- added joint Torso_BR: type revolute, parent Torso, child BR, origin xyz=0.5 -0.9 1 rpy=0 0 0, axis 1 0 0, limit lower=-3.14159 upper=3.14159 effort=0.0 velocity=0.0
- added joint Torso_BW: type revolute, parent Torso, child BW, origin xyz=0 -1 1 rpy=0 0 0, axis 1 0 0, limit lower=-3.14159 upper=3.14159 effort=0.0 velocity=0.0
- added joint Torso_FL: type revolute, parent Torso, child FL, origin xyz=-0.5 0.9 1 rpy=0 0 0, axis 1 0 0, limit lower=-3.14159 upper=3.14159 effort=0.0 velocity=0.0
- added joint Torso_FR: type revolute, parent Torso, child FR, origin xyz=0.5 0.9 1 rpy=0 0 0, axis 1 0 0, limit lower=-3.14159 upper=3.14159 effort=0.0 velocity=0.0
